File: kicad/Grow1x8/Grow1x8.kicad_pcb (KiCad board)
At the start: 2 copper layers, 77 x 24.5 mm, 3 parts, among them J1 Screw_Terminal_01x02, J2 Screw_Terminal_01x02

Commit message: latest
Parts:
- removed U1: ~, dlaw:LED 5630
- added L1: ~, dlaw:LED 5630, F.Cu at (90.2, 53.8)
- added L2: ~, dlaw:LED 5630, F.Cu at (109.9, 53.8)
- added L3: ~, dlaw:LED 5630, F.Cu at (129.7, 53.8)
- added L4: ~, dlaw:LED 5630, F.Cu at (149.5, 53.8)
- added L5: ~, dlaw:LED 5630, F.Cu at (169.2, 53.8)
- added L6: ~, dlaw:LED 5630, F.Cu at (189.0, 53.8)
- added L7: ~, dlaw:LED 5630, F.Cu at (208.7, 53.8)
- added L8: ~, dlaw:LED 5630, F.Cu at (228.5, 53.8)
- moved J2 120.8 mm to (250.5, 51.0)
- moved J1 8.27 mm to (70.0, 50.5)
Routing:
- net GND: track 51.6 -> 180.7 mm
- net +3.3V: track 51.6 -> 180.7 mm
Other:
- board size 77 x 24.5 mm -> 200 x 20 mm

Commit message: latest
Parts:
- moved L8 7.21 mm to (235.7, 54.3)
- moved L7 6.52 mm to (215.2, 54.3)
- moved L6 5.82 mm to (194.8, 54.3)
- moved L5 5.12 mm to (174.3, 54.3)
- moved L4 4.43 mm to (153.9, 54.3)
- moved L3 3.74 mm to (133.4, 54.3)
- moved L2 3.04 mm to (113.0, 54.3)
- moved L1 2.36 mm to (92.5, 54.3)
- moved J1 0.50 mm to (70.0, 51.0)
Routing:
- net +3.3V: track 180.7 -> 181.2 mm
Other:
- board text added: "corvidae v0.01"
