File: kicad/Grow1x8/Grow1x8.kicad_sch (KiCad schematic)
At the start: 3 parts, among them J1 Screw_Terminal_01x02, J2 Screw_Terminal_01x02

Commit message: latest
Parts:
- removed U1: ~, dlaw:LED 5630, symbol WaldLibs:LedTest
- added L1, L2, L3, L4, L5, L6, L7, L8: ~, dlaw:LED 5630, symbol WaldLibs:LedTest
Connections:
- net +3.3V: now also L1.1 (VCD), L2.1 (VCD), L3.1 (VCD), L4.1 (VCD), L5.1 (VCD), L6.1 (VCD), L7.1 (VCD), L8.1 (VCD)
- net GND: now also L1.3 (GND), L2.3 (GND), L3.3 (GND), L4.3 (GND), L5.3 (GND), L6.3 (GND), L7.3 (GND), L8.3 (GND)

Commit message: latest
Parts:
- removed L1, L2, L3, L4, L5, L6, L7, L8: ~, dlaw:LED 5630, symbol WaldLibs:LedTest
- added L1, L2, L3, L4, L5, L6, L7, L8: ~, dlaw:LED 5630, symbol dlaw:dlaw 5630
Connections:
- net +3.3V: now also L1.1 (VCD), L2.1 (VCD), L3.1 (VCD), L4.1 (VCD), L5.1 (VCD), L6.1 (VCD), L7.1 (VCD), L8.1 (VCD)
- net GND: now also L1.3 (GND), L2.3 (GND), L3.3 (GND), L4.3 (GND), L5.3 (GND), L6.3 (GND), L7.3 (GND), L8.3 (GND)
